Commit message: ROS2 Humble

File: xacro/depthcam.xacro (robot description, xacro)
@@ -31,5 +31,5 @@
         <origin xyz="${d435_cam_mount_from_center_offset} ${-d435_cam_depth_py} 0" rpy="${pi/2} 0 ${pi/2}"/>
         <geometry>
-          <mesh filename="package://realsense_ros_gazebo/meshes/realsense_d435.stl" />
+          <mesh filename="file://$(find realsense_ros_gazebo)/meshes/realsense_d435.stl" />
         </geometry>
       </visual>
@@ -230,5 +230,5 @@
               <origin rpy="0 0 0" xyz="0 0 0"/>
               <geometry>
-                  <mesh filename="package://realsense_ros_gazebo/meshes/realsense_r200/meshes/realsense.dae"/>
+                  <mesh filename="file://$(find realsense_ros_gazebo)/meshes/realsense_r200/meshes/realsense.dae"/>
               </geometry>
           </visual>

File: xacro/tracker.xacro (robot description, xacro)
@@ -90,5 +90,5 @@
             <origin rpy="1.57 0 1.57" xyz="0 0 0"/>
             <geometry>
-                <mesh filename="package://realsense_ros_gazebo/meshes/realsense_t265.stl" scale="0.001 0.001 0.001"/>
+                <mesh filename="file://$(find realsense_ros_gazebo)/meshes/realsense_t265.stl" scale="0.001 0.001 0.001"/>
             </geometry>
         </visual>

Commit message: D435 is 72 grams

File: xacro/depthcam.xacro (robot description, xacro)
@@ -10,5 +10,5 @@
     <xacro:property name="d435_cam_height" value="0.025"/>
     <xacro:property name="d435_cam_depth" value="0.02505"/>
-    <xacro:property name="d435_cam_mass" value="0.564"/>
+    <xacro:property name="d435_cam_mass" value="0.072"/>
     <xacro:property name="d435_cam_mount_from_center_offset" value="0.0149"/>
     <xacro:property name="d435_cam_depth_px" value="${d435_cam_mount_from_center_offset}"/>
